Commit message: feat: initial minimal launch start

File: src/auto_nav_part3/simulation/urdf/pioneer.urdf (robot description, URDF)
Before this commit: robot pioneer3at_body, 19 links, 18 joints
Links:
- removed link auto_nav/simulation_back_left_axle
- removed link auto_nav/simulation_back_left_hub
- removed link auto_nav/simulation_back_left_wheel
- removed link auto_nav/simulation_back_right_axle
- removed link auto_nav/simulation_back_right_hub
- removed link auto_nav/simulation_back_right_wheel
- removed link auto_nav/simulation_front_left_axle
- removed link auto_nav/simulation_front_left_hub
- removed link auto_nav/simulation_front_left_wheel
- removed link auto_nav/simulation_front_right_axle
- removed link auto_nav/simulation_front_right_hub
- removed link auto_nav/simulation_front_right_wheel
- added link auto_nav_part3/simulation_back_left_axle, mass 0.1; collision box size=0.01 0.01 0.01; visual mesh filename=package://auto_nav_part3/simulation/meshes/axle.dae
- added link auto_nav_part3/simulation_back_left_hub, mass 0.1; collision box size=0.01 0.01 0.01; visual mesh filename=package://auto_nav_part3/simulation/meshes/left_hubcap.dae
- added link auto_nav_part3/simulation_back_left_wheel, mass 0.5; collision cylinder length=0.075 radius=0.111; visual mesh filename=package://auto_nav_part3/simulation/meshes/wheel.dae
- added link auto_nav_part3/simulation_back_right_axle, mass 0.1; collision box size=0.01 0.01 0.01; visual mesh filename=package://auto_nav_part3/simulation/meshes/axle.dae
- added link auto_nav_part3/simulation_back_right_hub, mass 0.1; collision box size=0.01 0.01 0.01; visual mesh filename=package://auto_nav_part3/simulation/meshes/right_hubcap.dae
- added link auto_nav_part3/simulation_back_right_wheel, mass 0.5; collision cylinder length=0.075 radius=0.111; visual mesh filename=package://auto_nav_part3/simulation/meshes/wheel.dae
- added link auto_nav_part3/simulation_front_left_axle, mass 0.1; collision box size=0.01 0.01 0.01; visual mesh filename=package://auto_nav_part3/simulation/meshes/axle.dae
- added link auto_nav_part3/simulation_front_left_hub, mass 0.1; collision box size=0.01 0.01 0.01; visual mesh filename=package://auto_nav_part3/simulation/meshes/left_hubcap.dae
- added link auto_nav_part3/simulation_front_left_wheel, mass 0.5; collision cylinder length=0.075 radius=0.111; visual mesh filename=package://auto_nav_part3/simulation/meshes/wheel.dae
- added link auto_nav_part3/simulation_front_right_axle, mass 0.1; collision box size=0.01 0.01 0.01; visual mesh filename=package://auto_nav_part3/simulation/meshes/axle.dae
- added link auto_nav_part3/simulation_front_right_hub, mass 0.1; collision box size=0.01 0.01 0.01; visual mesh filename=package://auto_nav_part3/simulation/meshes/right_hubcap.dae
- added link auto_nav_part3/simulation_front_right_wheel, mass 0.5; collision cylinder length=0.075 radius=0.111; visual mesh filename=package://auto_nav_part3/simulation/meshes/wheel.dae
- link chassis: geometry collision mesh filename=package://auto_nav_part3/simulation/meshes/chassis.dae; visual mesh filename=package://auto_nav_part3/simulation/meshes/chassis.dae
- link laser_frame: geometry collision box size=0.01 0.01 0.01; visual mesh filename=package://auto_nav_part3/simulation/meshes/hokuyo1.dae
- link top_plate: geometry collision box size=0.1 0.1 0.1; visual mesh filename=package://auto_nav_part3/simulation/meshes/top.dae
Joints:
- removed joint auto_nav/simulation_back_left_wheel_joint
- removed joint auto_nav/simulation_back_right_wheel_joint
- removed joint auto_nav/simulation_front_left_wheel_joint
- removed joint auto_nav/simulation_front_right_wheel_joint
- added joint auto_nav_part3/simulation_back_left_wheel_joint: type continuous, parent auto_nav_part3/simulation_back_left_hub, child auto_nav_part3/simulation_back_left_wheel, origin xyz=0 0 0 rpy=0 0 0, axis 0 1 0, limit effort=100 velocity=100
- added joint auto_nav_part3/simulation_back_right_wheel_joint: type continuous, parent auto_nav_part3/simulation_back_right_hub, child auto_nav_part3/simulation_back_right_wheel, origin xyz=0 0 0 rpy=0 0 0, axis 0 1 0, limit effort=100 velocity=100
- added joint auto_nav_part3/simulation_front_left_wheel_joint: type continuous, parent auto_nav_part3/simulation_front_left_hub, child auto_nav_part3/simulation_front_left_wheel, origin xyz=0 0 0 rpy=0 0 0, axis 0 1 0, limit effort=100 velocity=100
- added joint auto_nav_part3/simulation_front_right_wheel_joint: type continuous, parent auto_nav_part3/simulation_front_right_hub, child auto_nav_part3/simulation_front_right_wheel, origin xyz=0 0 0 rpy=0 0 0, axis 0 1 0, limit effort=100 velocity=100
- joint base_back_left_axle_joint: child auto_nav/simulation_back_left_axle -> auto_nav_part3/simulation_back_left_axle
- joint base_back_left_hub_joint: child auto_nav/simulation_back_left_hub -> auto_nav_part3/simulation_back_left_hub; parent auto_nav/simulation_back_left_axle -> auto_nav_part3/simulation_back_left_axle
- joint base_back_right_axle_joint: child auto_nav/simulation_back_right_axle -> auto_nav_part3/simulation_back_right_axle
- joint base_back_right_hub_joint: child auto_nav/simulation_back_right_hub -> auto_nav_part3/simulation_back_right_hub; parent auto_nav/simulation_back_right_axle -> auto_nav_part3/simulation_back_right_axle
- joint base_front_left_axle_joint: child auto_nav/simulation_front_left_axle -> auto_nav_part3/simulation_front_left_axle
- joint base_front_left_hub_joint: child auto_nav/simulation_front_left_hub -> auto_nav_part3/simulation_front_left_hub; parent auto_nav/simulation_front_left_axle -> auto_nav_part3/simulation_front_left_axle
- joint base_front_right_axle_joint: child auto_nav/simulation_front_right_axle -> auto_nav_part3/simulation_front_right_axle
- joint base_front_right_hub_joint: child auto_nav/simulation_front_right_hub -> auto_nav_part3/simulation_front_right_hub; parent auto_nav/simulation_front_right_axle -> auto_nav_part3/simulation_front_right_axle
