Commit message: feat: configure Gazebo sim and RViz2 for Pioneer 3-AT
- Add sim_bringup.launch.py: launches Gazebo server+GUI separately to
  prevent cascade shutdown; server uses --headless-rendering and ogre
  render engine to avoid SIGSEGV from camera/lidar sensors on ARM/VM;
  GUI uses ogre to avoid ogre2 crash on Parallels Apple Silicon
- Fix mesh display: OpaqueFunction pre-processes URDF at launch time,
  replacing package:// URIs with file:// absolute paths so Gazebo's
  gz-common5-graphics mesh loader can find .dae files
- Add discovery_15x15.sdf world: 15x15m arena with white boundary lines,
  Sensors plugin set to ogre render engine for ARM stability
- Spawn pioneer at bottom-centre (x=0, y=-6.5) facing positive-Y
- Add joint_state_publisher so wheel joints have states for RSP/RViz2
- Add pioneer.rviz: Fixed Frame=base_link, Transient Local QoS on
  /robot_description, TF and RobotModel displays configured
- Add scripts/launch.sh: build/source/run wrapper with list and start
  subcommands; sets LIBGL_ALWAYS_SOFTWARE and QT_OPENGL=software for
  VM software rendering
- Relocate simulation assets (urdf, meshes, worlds) into the Python
  package directory so setup.py installs them to the share path
- Fix URDF bugs: remove invalid geometry name= attribute, replace
  joint_properties with dynamics, remove anchor elements, update
  JointStatePublisher plugin name to gz:: namespace

File: src/auto_nav_part3/auto_nav_part3/simulation/urdf/pioneer.urdf (robot description, URDF)
Before this commit: robot pioneer3at_body, 19 links, 18 joints
Links:
- removed link auto_nav_part3/simulation_back_left_axle
- removed link auto_nav_part3/simulation_back_left_hub
- removed link auto_nav_part3/simulation_back_left_wheel
- removed link auto_nav_part3/simulation_back_right_axle
- removed link auto_nav_part3/simulation_back_right_hub
- removed link auto_nav_part3/simulation_back_right_wheel
- removed link auto_nav_part3/simulation_front_left_axle
- removed link auto_nav_part3/simulation_front_left_hub
- removed link auto_nav_part3/simulation_front_left_wheel
- removed link auto_nav_part3/simulation_front_right_axle
- removed link auto_nav_part3/simulation_front_right_hub
- removed link auto_nav_part3/simulation_front_right_wheel
- added link back_left_axle, mass 0.1; collision box size=0.01 0.01 0.01; visual mesh filename=package://auto_nav_part3/simulation/meshes/axle.dae
- added link back_left_hub, mass 0.1; collision box size=0.01 0.01 0.01; visual mesh filename=package://auto_nav_part3/simulation/meshes/left_hubcap.dae
- added link back_left_wheel, mass 0.5; collision cylinder length=0.075 radius=0.111; visual mesh filename=package://auto_nav_part3/simulation/meshes/wheel.dae
- added link back_right_axle, mass 0.1; collision box size=0.01 0.01 0.01; visual mesh filename=package://auto_nav_part3/simulation/meshes/axle.dae
- added link back_right_hub, mass 0.1; collision box size=0.01 0.01 0.01; visual mesh filename=package://auto_nav_part3/simulation/meshes/right_hubcap.dae
- added link back_right_wheel, mass 0.5; collision cylinder length=0.075 radius=0.111; visual mesh filename=package://auto_nav_part3/simulation/meshes/wheel.dae
- added link front_left_axle, mass 0.1; collision box size=0.01 0.01 0.01; visual mesh filename=package://auto_nav_part3/simulation/meshes/axle.dae
- added link front_left_hub, mass 0.1; collision box size=0.01 0.01 0.01; visual mesh filename=package://auto_nav_part3/simulation/meshes/left_hubcap.dae
- added link front_left_wheel, mass 0.5; collision cylinder length=0.075 radius=0.111; visual mesh filename=package://auto_nav_part3/simulation/meshes/wheel.dae
- added link front_right_axle, mass 0.1; collision box size=0.01 0.01 0.01; visual mesh filename=package://auto_nav_part3/simulation/meshes/axle.dae
- added link front_right_hub, mass 0.1; collision box size=0.01 0.01 0.01; visual mesh filename=package://auto_nav_part3/simulation/meshes/right_hubcap.dae
- added link front_right_wheel, mass 0.5; collision cylinder length=0.075 radius=0.111; visual mesh filename=package://auto_nav_part3/simulation/meshes/wheel.dae
Joints:
- removed joint auto_nav_part3/simulation_back_left_wheel_joint
- removed joint auto_nav_part3/simulation_back_right_wheel_joint
- removed joint auto_nav_part3/simulation_front_left_wheel_joint
- removed joint auto_nav_part3/simulation_front_right_wheel_joint
- added joint back_left_wheel_joint: type continuous, parent back_left_hub, child back_left_wheel, origin xyz=0 0 0 rpy=0 0 0, axis 0 1 0, limit effort=100 velocity=100
- added joint back_right_wheel_joint: type continuous, parent back_right_hub, child back_right_wheel, origin xyz=0 0 0 rpy=0 0 0, axis 0 1 0, limit effort=100 velocity=100
- added joint front_left_wheel_joint: type continuous, parent front_left_hub, child front_left_wheel, origin xyz=0 0 0 rpy=0 0 0, axis 0 1 0, limit effort=100 velocity=100
- added joint front_right_wheel_joint: type continuous, parent front_right_hub, child front_right_wheel, origin xyz=0 0 0 rpy=0 0 0, axis 0 1 0, limit effort=100 velocity=100
- joint base_back_left_axle_joint: child auto_nav_part3/simulation_back_left_axle -> back_left_axle
- joint base_back_left_hub_joint: child auto_nav_part3/simulation_back_left_hub -> back_left_hub; parent auto_nav_part3/simulation_back_left_axle -> back_left_axle
- joint base_back_right_axle_joint: child auto_nav_part3/simulation_back_right_axle -> back_right_axle
- joint base_back_right_hub_joint: child auto_nav_part3/simulation_back_right_hub -> back_right_hub; parent auto_nav_part3/simulation_back_right_axle -> back_right_axle
- joint base_front_left_axle_joint: child auto_nav_part3/simulation_front_left_axle -> front_left_axle
- joint base_front_left_hub_joint: child auto_nav_part3/simulation_front_left_hub -> front_left_hub; parent auto_nav_part3/simulation_front_left_axle -> front_left_axle
- joint base_front_right_axle_joint: child auto_nav_part3/simulation_front_right_axle -> front_right_axle
- joint base_front_right_hub_joint: child auto_nav_part3/simulation_front_right_hub -> front_right_hub; parent auto_nav_part3/simulation_front_right_axle -> front_right_axle
